Commit message: fix: change the arm for SAR and fix it in sim

File: urc_hw_description/urdf/drivebase.xacro (robot description, xacro)
@@ -23,4 +23,9 @@
     </xacro:macro> -->
     <xacro:macro name="drivebase" params="wheel_radius wheel_thickness wheel_friction approximate">
+        <link name="world" />
+        <joint name="fixed" type="fixed">
+            <parent link="world" />
+            <child link="base_link" />
+        </joint>
         <link name="base_link">
             <inertial>
